File: design/esp-light-controller/esp-light-controller.kicad_pcb (KiCad board)
At the start: 4 copper layers, 50 x 57.6 mm, 48 parts, among them J1 LED0, J2 LED1, J3 LED2, J4 PWM_FAN, P1 USB_C_Plug_USB2.0, Q1 2N7002, Q2 2N7002, Q3 2N7002, Q4 2N7002, Q5 2N7002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

Commit message: rev e
Parts:
- removed J4: PWM_FAN, Connector_PinHeader_2.54mm:PinHeader_1x04_P2.54mm_Vertical
- added FAN: FAN, Connector_PinHeader_2.54mm:PinHeader_1x04_P2.54mm_Vertical, F.Cu at (117.2, 68.6)
- added J5: IO, Connector_PinHeader_2.54mm:PinHeader_2x04_P2.54mm_Vertical, F.Cu at (160.5, 68.8)
- added R18: 4.7k, Resistor_SMD:R_0805_2012Metric, F.Cu at (128.1, 87.8)
- added TP1: temp, TestPoint:TestPoint_Pad_1.5x1.5mm, F.Cu at (125.7, 77.7)
- added TP2: fan(16), TestPoint:TestPoint_Pad_1.5x1.5mm, F.Cu at (120.4, 68.6)
- added TP3: dtr, TestPoint:TestPoint_Pad_1.5x1.5mm, F.Cu at (134.1, 78.4)
- added TP4: rts, TestPoint:TestPoint_Pad_1.5x1.5mm, F.Cu at (138.8, 78.5)
- added TP5: tach(17), TestPoint:TestPoint_Pad_1.5x1.5mm, F.Cu at (120.4, 71.2)
- G***: moved to B.Cu
- moved C5 43.9 mm to (118.0, 86.2), turned to 0 degrees
- moved C3 42.5 mm to (121.5, 86.2), turned to 180 degrees
- moved U4 35.4 mm to (127.1, 82.8), turned to 90 degrees
- moved G*** 16.6 mm to (140.1, 73.4), turned to 180 degrees
- moved C1 0.13 mm to (135.3, 90.2)
Connections:
- U3 pad 10: unconnected-(U3-Pad10) -> /io25
- U3 pad 11: unconnected-(U3-Pad11) -> /io26
- U3 pad 33: unconnected-(U3-Pad33) -> /sda
- U3 pad 36: unconnected-(U3-Pad36) -> /scl
- U3 pad 37: unconnected-(U3-Pad37) -> /io23
Routing:
- net /scl: track 0.00 -> 42.6 mm, vias 0 -> 2
- net /io23: track 0.00 -> 39.1 mm, vias 0 -> 1
- net /sda: track 0.00 -> 38.5 mm, vias 0 -> 1
- net /fanctl: track 30.1 -> 47.1 mm
- net /io25: track 0.00 -> 14.9 mm
- net /io26: track 0.00 -> 13.3 mm
- net /dtr: track 16.4 -> 28.1 mm, vias 2 -> 4
- net Net-(R18-Pad2): track 23.8 -> 32.6 mm
- net +3V3: track 56.3 -> 62.5 mm, vias 14 -> 11
- net /rts: track 19.7 -> 25.7 mm, vias 2 -> 4
- net /ledctl0: track 39.1 -> 34.5 mm, vias 2 -> 0
- net /tach: track 36.7 -> 40.8 mm
- net /ledctl1: track 35.7 -> 33.7 mm
- net /en: track 77.9 -> 76.9 mm
- net +5V: track 42.3 -> 42.9 mm
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Other:
- board text added: "- + 13"
- board text added: "- + 14"
- board text added: "- + 15"
- board text added: "23"
- board text added: "25"
- board text added: "26"
- board text added: "3V3"
- board text added: "5V"
- board text added: "5V GND"
- board text added: "GND"
- board text added: "SCL"
- board text added: "SDA"
- board text added: "helios :: Rev E nnarain"
- board text removed: "- + >"
- board text removed: "FAN TACH 5V GND"
- board text removed: "helios :: Rev D nnarain"
