File: design/esp-light-controller/esp-light-controller.kicad_sch (KiCad schematic)
At the start: 45 parts, among them J1 LED0, J2 LED1, J3 LED2, J4 PWM_FAN, P1 USB_C_Plug_USB2.0, Q1 2N7002, Q2 2N7002, Q3 2N7002, Q4 2N7002, Q5 2N7002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

Commit message: rev e
Parts:
- added J5: IO, Connector_PinHeader_2.54mm:PinHeader_2x04_P2.54mm_Vertical, symbol Connector_Generic:Conn_02x04_Odd_Even
- added R18: 4.7k, Resistor_SMD:R_0805_2012Metric, symbol Device:R
- added TP1: temp, TestPoint:TestPoint_Pad_1.5x1.5mm, symbol Connector:TestPoint
- added TP2: fan, TestPoint:TestPoint_Pad_1.5x1.5mm, symbol Connector:TestPoint
- added TP3: dtr, TestPoint:TestPoint_Pad_1.5x1.5mm, symbol Connector:TestPoint
- added TP4: rts, TestPoint:TestPoint_Pad_1.5x1.5mm, symbol Connector:TestPoint
- added TP5: tach, TestPoint:TestPoint_Pad_1.5x1.5mm, symbol Connector:TestPoint
- J4: value PWM_FAN -> FAN
Connections:
- net +3V3: now also J5.3 (Pin_3), R18.1
- net +5V: now also J5.1 (Pin_1)
- net GND: now also J5.5 (Pin_5)
- net dtr: now also TP3.1
- net fanctl: now also TP2.1
- net rts: now also TP4.1
- net tach: now also TP5.1
- net at U3.30 (IO18), U4.4 (DQ): now also R18.2, TP1.1
- net io25: now reaches U3.10 (IO25)
- net io25: now also J5.8 (Pin_8)
- net io26: now reaches U3.11 (IO26)
- net io26: now also J5.7 (Pin_7)
- net sda: now reaches U3.33 (IO21)
- net sda: now also J5.4 (Pin_4)
- net scl: now reaches U3.36 (IO22)
- net scl: now also J5.2 (Pin_2)
- net io23: now reaches U3.37 (IO23)
- net io23: now also J5.6 (Pin_6)
Other:
- note added: "Fan / I2C / DIO"
- note added: "Temperature Sensor"
- note removed: "Fan / Temperature Control"
- title: ESP Light Controller -> Helios Light Controller
- moved on the sheet: C10, C8, C9, J1, J2, J3, R13, R14, R15, U4
